Commit message: Integrate AR4-MK3 model, add camera tower obstacle, and configure MoveIt2

File: ros2_ws/src/james_description/urdf/james.urdf.xacro (robot description, xacro)
@@ -1,4 +1,7 @@
 <?xml version="1.0"?>
 <robot xmlns:xacro="http://www.ros.org/wiki/xacro" name="james">
+  <!-- Include AR4 Macro -->
+  <xacro:include filename="$(find james_description)/urdf/ar4/ar_macro.xacro" />
+  <!-- Base Link (Platform) -->
   <link name="base_link">
     <visual>
@@ -10,4 +13,71 @@
       </material>
     </visual>
+    <collision>
+      <geometry>
+        <box size="0.45 0.56 0.1"/>
+      </geometry>
+    </collision>
+    <inertial>
+      <mass value="20.0"/>
+      <origin xyz="0 0 0" rpy="0 0 0"/>
+      <inertia ixx="0.5" ixy="0" ixz="0" iyy="0.5" iyz="0" izz="0.5"/>
+    </inertial>
   </link>
+  <link name="base_footprint"/>
+  <joint name="base_footprint_joint" type="fixed">
+    <parent link="base_footprint"/>
+    <child link="base_link"/>
+    <origin xyz="0 0 0.1" rpy="0 0 0"/> <!-- Assumed platform height above ground -->
+  </joint>
+  <!-- Camera Tower (Obstacle/Camera Mount) -->
+  <link name="camera_tower_link">
+    <visual>
+      <origin xyz="0 0 0.6" rpy="0 0 0"/>
+      <geometry>
+        <box size="0.04 0.04 1.2"/>
+      </geometry>
+      <material name="silver">
+        <color rgba="0.75 0.75 0.75 1"/>
+      </material>
+    </visual>
+    <collision>
+      <origin xyz="0 0 0.6" rpy="0 0 0"/>
+      <geometry>
+        <box size="0.04 0.04 1.2"/>
+      </geometry>
+    </collision>
+    <inertial>
+      <mass value="2.0"/>
+      <origin xyz="0 0 0.6" rpy="0 0 0"/>
+      <inertia ixx="0.2" ixy="0" ixz="0" iyy="0.2" iyz="0" izz="0.01"/>
+    </inertial>
+  </link>
+  <joint name="camera_tower_joint" type="fixed">
+    <parent link="base_link"/>
+    <child link="camera_tower_link"/>
+    <origin xyz="-0.2 0 0.05" rpy="0 0 0"/> <!-- Positioned at back of base -->
+  </joint>
+  <!-- Instantiate AR4 Robot Arm -->
+  <xacro:ar_robot
+    tf_prefix="arm_"
+    parent="base_link"
+    robot_parameters_file="$(find james_description)/config/ar4_custom_limits.yaml">
+    <origin xyz="0.15 0 0.05" rpy="0 0 0" /> <!-- Mounted at front-center of base -->
+  </xacro:ar_robot>
+  <!-- Custom Gripper (Placeholder) -->
+  <link name="gripper_link">
+    <visual>
+      <geometry>
+        <box size="0.05 0.08 0.1"/>
+      </geometry>
+      <material name="grey">
+        <color rgba="0.5 0.5 0.5 1"/>
+      </material>
+    </visual>
+  </link>
+  <joint name="gripper_joint" type="fixed">
+    <parent link="arm_ee_link"/>
+    <child link="gripper_link"/>
+    <origin xyz="0 0 0.05" rpy="0 0 0"/>
+  </joint>
 </robot>

Commit message: Rviz to the rescue - arm definition refined

File: ros2_ws/src/james_description/urdf/james.urdf.xacro (robot description, xacro)
@@ -56,5 +56,5 @@
     <parent link="base_link"/>
     <child link="camera_tower_link"/>
-    <origin xyz="-0.2 0 0.05" rpy="0 0 0"/> <!-- Positioned at back of base -->
+    <origin xyz="0 0.35 0.05" rpy="0 0 0"/> <!-- Positioned at back of base (Y+) -->
   </joint>
   <!-- Instantiate AR4 Robot Arm -->
@@ -75,4 +75,9 @@
       </material>
     </visual>
+    <collision>
+      <geometry>
+        <box size="0.05 0.08 0.1"/>
+      </geometry>
+    </collision>
   </link>
   <joint name="gripper_joint" type="fixed">

Commit message: updatin robot definition and intelligent logging

File: ros2_ws/src/james_description/urdf/james.urdf.xacro (robot description, xacro)
@@ -63,5 +63,5 @@
     parent="base_link"
     robot_parameters_file="$(find james_description)/config/ar4_custom_limits.yaml">
-    <origin xyz="0.15 0 0.05" rpy="0 0 0" /> <!-- Mounted at front-center of base -->
+    <origin xyz="0.15 0 0.05" rpy="0 0 -1.5708" /> <!-- Rotated 90 deg to align J1=0 with Forward axis -->
   </xacro:ar_robot>
   <!-- Custom Gripper (Placeholder) -->

Commit message: updatin robot definition and intelligent logging2

File: ros2_ws/src/james_description/urdf/james.urdf.xacro (robot description, xacro)
@@ -63,5 +63,5 @@
     parent="base_link"
     robot_parameters_file="$(find james_description)/config/ar4_custom_limits.yaml">
-    <origin xyz="0.15 0 0.05" rpy="0 0 -1.5708" /> <!-- Rotated 90 deg to align J1=0 with Forward axis -->
+    <origin xyz="0.15 0 0.05" rpy="0 0 -1.5708" /> <!-- Standard ROS: Arm J1=0 points Forward (+X) -->
   </xacro:ar_robot>
   <!-- Custom Gripper (Placeholder) -->

Commit message: updatin robot definition and intelligent logging2

File: ros2_ws/src/james_description/urdf/james.urdf.xacro (robot description, xacro)
@@ -56,5 +56,5 @@
     <parent link="base_link"/>
     <child link="camera_tower_link"/>
-    <origin xyz="0 0.35 0.05" rpy="0 0 0"/> <!-- Positioned at back of base (Y+) -->
+    <origin xyz="0 -0.35 0.05" rpy="0 0 0"/> <!-- Positioned at back of base (Y-) -->
   </joint>
   <!-- Instantiate AR4 Robot Arm -->
@@ -63,5 +63,5 @@
     parent="base_link"
     robot_parameters_file="$(find james_description)/config/ar4_custom_limits.yaml">
-    <origin xyz="0.15 0 0.05" rpy="0 0 -1.5708" /> <!-- Standard ROS: Arm J1=0 points Forward (+X) -->
+    <origin xyz="0.15 0 0.05" rpy="0 0 3.14159" /> <!-- Facing +Y (Forward) -->
   </xacro:ar_robot>
   <!-- Custom Gripper (Placeholder) -->

Commit message: updatin robot definition

File: ros2_ws/src/james_description/urdf/james.urdf.xacro (robot description, xacro)
@@ -63,5 +63,5 @@
     parent="base_link"
     robot_parameters_file="$(find james_description)/config/ar4_custom_limits.yaml">
-    <origin xyz="0.15 0 0.05" rpy="0 0 3.14159" /> <!-- Facing +Y (Forward) -->
+    <origin xyz="0.15 0 0.05" rpy="0 0 3.1415926" /> <!-- Forward is now +Y -->
   </xacro:ar_robot>
   <!-- Custom Gripper (Placeholder) -->

Commit message: continuous debugging

File: ros2_ws/src/james_description/urdf/james.urdf.xacro (robot description, xacro)
@@ -56,5 +56,5 @@
     <parent link="base_link"/>
     <child link="camera_tower_link"/>
-    <origin xyz="0 -0.35 0.05" rpy="0 0 0"/> <!-- Positioned at back of base (Y-) -->
+    <origin xyz="0 0.35 0.05" rpy="0 0 0"/> <!-- Positioned at back of base (Y+) -->
   </joint>
   <!-- Instantiate AR4 Robot Arm -->
@@ -63,5 +63,5 @@
     parent="base_link"
     robot_parameters_file="$(find james_description)/config/ar4_custom_limits.yaml">
-    <origin xyz="0.15 0 0.05" rpy="0 0 3.1415926" /> <!-- Forward is now +Y -->
+    <origin xyz="0.15 0 0.05" rpy="0 0 0" /> <!-- Mounted at front-center of base -->
   </xacro:ar_robot>
   <!-- Custom Gripper (Placeholder) -->

Commit message: Implementing Kinematic Alignment and Joint Inversions

File: ros2_ws/src/james_description/urdf/james.urdf.xacro (robot description, xacro)
@@ -56,5 +56,5 @@
     <parent link="base_link"/>
     <child link="camera_tower_link"/>
-    <origin xyz="0 0.35 0.05" rpy="0 0 0"/> <!-- Positioned at back of base (Y+) -->
+    <origin xyz="0 -0.35 0.05" rpy="0 0 0"/> <!-- Positioned at back of base (Y-) -->
   </joint>
   <!-- Instantiate AR4 Robot Arm -->
@@ -63,5 +63,5 @@
     parent="base_link"
     robot_parameters_file="$(find james_description)/config/ar4_custom_limits.yaml">
-    <origin xyz="0.15 0 0.05" rpy="0 0 0" /> <!-- Mounted at front-center of base -->
+    <origin xyz="0.15 0 0.05" rpy="0 0 3.1415926" /> <!-- Forward is now +Y -->
   </xacro:ar_robot>
   <!-- Custom Gripper (Placeholder) -->
