Commit message: Fix xacro evaluation error for ROS2 Foxy

File: ros2_ws/src/james_description/urdf/ar4/ar_macro.xacro (robot description, xacro)
@@ -1,4 +1,4 @@
 <?xml version="1.0" encoding="utf-8"?>
-<robot xmlns:xacro="http://wiki.ros.org/xacro">
+<robot xmlns:xacro="http://www.ros.org/wiki/xacro">
   <xacro:macro name="ar_robot" params="
     tf_prefix
@@ -7,5 +7,5 @@
     robot_parameters_file
   ">
-    <xacro:property name="robot_parameters" value="${xacro.load_yaml(robot_parameters_file)}"/>
+    <xacro:property name="robot_parameters" value="${load_yaml(robot_parameters_file)}"/>
     <joint name="${tf_prefix}base_joint" type="fixed">
       <xacro:insert_block name="origin" />

Commit message: robot definition update

File: ros2_ws/src/james_description/urdf/ar4/ar_macro.xacro (robot description, xacro)
@@ -61,5 +61,5 @@
       <parent link="${tf_prefix}base_link"/>
       <child link="${tf_prefix}link_1"/>
-      <axis xyz="0 0 1"/>
+      <axis xyz="0 0 -1"/>
       <limit
         lower="${robot_parameters['j1_limit_min']}"

Commit message: swapping controller mapping again

File: ros2_ws/src/james_description/urdf/ar4/ar_macro.xacro (robot description, xacro)
@@ -61,5 +61,5 @@
       <parent link="${tf_prefix}base_link"/>
       <child link="${tf_prefix}link_1"/>
-      <axis xyz="0 0 -1"/>
+      <axis xyz="0 0 1"/>
       <limit
         lower="${robot_parameters['j1_limit_min']}"

Commit message: swapping controller mapping again

File: ros2_ws/src/james_description/urdf/ar4/ar_macro.xacro (robot description, xacro)
@@ -95,5 +95,5 @@
       <parent link="${tf_prefix}link_1"/>
       <child link="${tf_prefix}link_2"/>
-      <axis xyz="0 0 -1"/>
+      <axis xyz="0 0 1"/>
       <limit
         lower="${robot_parameters['j2_limit_min']}"

Commit message: Implementing Kinematic Alignment

File: ros2_ws/src/james_description/urdf/ar4/ar_macro.xacro (robot description, xacro)
@@ -58,5 +58,5 @@
     </link>
     <joint name="${tf_prefix}joint_1" type="revolute">
-      <origin rpy="${pi} 0 0" xyz="0 0 0"/>
+      <origin rpy="0 0 0" xyz="0 0 0"/>
       <parent link="${tf_prefix}base_link"/>
       <child link="${tf_prefix}link_1"/>

File: ros2_ws/src/james_description/urdf/james.urdf.xacro (robot description, xacro)
@@ -63,5 +63,5 @@
     parent="base_link"
     robot_parameters_file="$(find james_description)/config/ar4_custom_limits.yaml">
-    <origin xyz="0.15 0 0.05" rpy="0 0 3.1415926" /> <!-- Forward is now +Y -->
+    <origin xyz="0.15 0 0.05" rpy="0 0 1.5708" /> <!-- Forward is now +Y -->
   </xacro:ar_robot>
   <!-- Custom Gripper (Placeholder) -->

Commit message: more remodeling

File: ros2_ws/src/james_description/urdf/ar4/ar_macro.xacro (robot description, xacro)
@@ -58,8 +58,8 @@
     </link>
     <joint name="${tf_prefix}joint_1" type="revolute">
-      <origin rpy="0 0 0" xyz="0 0 0"/>
+      <origin rpy="${pi} 0 0" xyz="0 0 0"/>
       <parent link="${tf_prefix}base_link"/>
       <child link="${tf_prefix}link_1"/>
-      <axis xyz="0 0 1"/>
+      <axis xyz="0 0 -1"/>
       <limit
         lower="${robot_parameters['j1_limit_min']}"
@@ -95,5 +95,5 @@
       <parent link="${tf_prefix}link_1"/>
       <child link="${tf_prefix}link_2"/>
-      <axis xyz="0 0 1"/>
+      <axis xyz="0 0 -1"/>
       <limit
         lower="${robot_parameters['j2_limit_min']}"
@@ -129,5 +129,5 @@
       <parent link="${tf_prefix}link_2"/>
       <child link="${tf_prefix}link_3"/>
-      <axis xyz="0 0 -1"/>
+      <axis xyz="0 0 1"/>
       <limit
         lower="${robot_parameters['j3_limit_min']}"
@@ -163,5 +163,5 @@
       <parent link="${tf_prefix}link_3"/>
       <child link="${tf_prefix}link_4"/>
-      <axis xyz="0 0 -1"/>
+      <axis xyz="0 0 1"/>
       <limit
         lower="${robot_parameters['j4_limit_min']}"
@@ -231,5 +231,5 @@
       <parent link="${tf_prefix}link_5"/>
       <child link="${tf_prefix}link_6"/>
-      <axis xyz="0 0 1"/>
+      <axis xyz="0 0 -1"/>
       <limit
         lower="${robot_parameters['j6_limit_min']}"

Commit message: more remodeling again

File: ros2_ws/src/james_description/urdf/ar4/ar_macro.xacro (robot description, xacro)
@@ -95,5 +95,5 @@
       <parent link="${tf_prefix}link_1"/>
       <child link="${tf_prefix}link_2"/>
-      <axis xyz="0 0 -1"/>
+      <axis xyz="0 0 1"/>
       <limit
         lower="${robot_parameters['j2_limit_min']}"
@@ -129,5 +129,5 @@
       <parent link="${tf_prefix}link_2"/>
       <child link="${tf_prefix}link_3"/>
-      <axis xyz="0 0 1"/>
+      <axis xyz="0 0 -1"/>
       <limit
         lower="${robot_parameters['j3_limit_min']}"
@@ -163,5 +163,5 @@
       <parent link="${tf_prefix}link_3"/>
       <child link="${tf_prefix}link_4"/>
-      <axis xyz="0 0 1"/>
+      <axis xyz="0 0 -1"/>
       <limit
         lower="${robot_parameters['j4_limit_min']}"
@@ -231,5 +231,5 @@
       <parent link="${tf_prefix}link_5"/>
       <child link="${tf_prefix}link_6"/>
-      <axis xyz="0 0 -1"/>
+      <axis xyz="0 0 1"/>
       <limit
         lower="${robot_parameters['j6_limit_min']}"

File: ros2_ws/src/james_description/urdf/james.urdf.xacro (robot description, xacro)
@@ -63,5 +63,5 @@
     parent="base_link"
     robot_parameters_file="$(find james_description)/config/ar4_custom_limits.yaml">
-    <origin xyz="0.15 0 0.05" rpy="0 0 1.5708" /> <!-- Forward is now +Y -->
+    <origin xyz="0.15 0 0.05" rpy="0 0 0" /> <!-- Forward is now +Y -->
   </xacro:ar_robot>
   <!-- Custom Gripper (Placeholder) -->

Commit message: more remodeling until pose matches real life

File: ros2_ws/src/james_description/urdf/ar4/ar_macro.xacro (robot description, xacro)
@@ -129,5 +129,5 @@
       <parent link="${tf_prefix}link_2"/>
       <child link="${tf_prefix}link_3"/>
-      <axis xyz="0 0 -1"/>
+      <axis xyz="0 0 1"/>
       <limit
         lower="${robot_parameters['j3_limit_min']}"

File: ros2_ws/src/james_description/urdf/james.urdf.xacro (robot description, xacro)
@@ -63,5 +63,5 @@
     parent="base_link"
     robot_parameters_file="$(find james_description)/config/ar4_custom_limits.yaml">
-    <origin xyz="0.15 0 0.05" rpy="0 0 0" /> <!-- Forward is now +Y -->
+    <origin xyz="0.15 0 0.05" rpy="0 0 3.1415926" /> <!-- Forward is now +Y -->
   </xacro:ar_robot>
   <!-- Custom Gripper (Placeholder) -->

Commit message: more remodeling until pose matches real life

File: ros2_ws/src/james_description/urdf/ar4/ar_macro.xacro (robot description, xacro)
@@ -95,5 +95,5 @@
       <parent link="${tf_prefix}link_1"/>
       <child link="${tf_prefix}link_2"/>
-      <axis xyz="0 0 1"/>
+      <axis xyz="0 0 -1"/>
       <limit
         lower="${robot_parameters['j2_limit_min']}"
@@ -129,5 +129,5 @@
       <parent link="${tf_prefix}link_2"/>
       <child link="${tf_prefix}link_3"/>
-      <axis xyz="0 0 1"/>
+      <axis xyz="0 0 -1"/>
       <limit
         lower="${robot_parameters['j3_limit_min']}"
@@ -231,5 +231,5 @@
       <parent link="${tf_prefix}link_5"/>
       <child link="${tf_prefix}link_6"/>
-      <axis xyz="0 0 1"/>
+      <axis xyz="0 0 -1"/>
       <limit
         lower="${robot_parameters['j6_limit_min']}"
