Commit message: simplifying IK by building groups

File: ros2_ws/src/james_description/srdf/ar_macro.srdf.xacro (robot description, xacro)
@@ -12,4 +12,17 @@
       <joint name="${tf_prefix}joint_4" />
       <joint name="${tf_prefix}joint_5" />
+      <joint name="${tf_prefix}joint_6" />
+      <joint name="${tf_prefix}ee_joint"/>
+    </group>
+    <!-- Sub-group for stable cartesian translation (X, Y, Z). Locks J4 and J6. -->
+    <group name="ar_translator">
+      <joint name="${tf_prefix}joint_1" />
+      <joint name="${tf_prefix}joint_2" />
+      <joint name="${tf_prefix}joint_3" />
+      <joint name="${tf_prefix}joint_5" />
+      <joint name="${tf_prefix}ee_joint"/>
+    </group>
+    <!-- Sub-group for wrist-only control. -->
+    <group name="ar_wrist">
       <joint name="${tf_prefix}joint_6" />
       <joint name="${tf_prefix}ee_joint"/>

Commit message: simplifying IK by building groupsV4

File: ros2_ws/src/james_description/srdf/ar_macro.srdf.xacro (robot description, xacro)
@@ -17,10 +17,12 @@
     <!-- Sub-group for stable cartesian translation (X, Y, Z). Locks J4 and J6. -->
     <group name="ar_translator">
-      <joint name="${tf_prefix}joint_1" />
-      <joint name="${tf_prefix}joint_2" />
-      <joint name="${tf_prefix}joint_3" />
-      <joint name="${tf_prefix}joint_5" />
-      <joint name="${tf_prefix}ee_joint"/>
-    </group>
+    <joint name="${tf_prefix}joint_1" />
+    <joint name="${tf_prefix}joint_2" />
+    <joint name="${tf_prefix}joint_3" />
+    <joint name="${tf_prefix}joint_4" />
+    <joint name="${tf_prefix}joint_5" />
+    <joint name="${tf_prefix}joint_6" />
+    <joint name="${tf_prefix}ee_joint" />
+  </group>
     <!-- Sub-group for wrist-only control. -->
     <group name="ar_wrist">

Commit message: simplifying IK by building groupsV5

File: ros2_ws/src/james_description/srdf/ar_macro.srdf.xacro (robot description, xacro)
@@ -17,16 +17,9 @@
     <!-- Sub-group for stable cartesian translation (X, Y, Z). Locks J4 and J6. -->
     <group name="ar_translator">
-    <joint name="${tf_prefix}joint_1" />
-    <joint name="${tf_prefix}joint_2" />
-    <joint name="${tf_prefix}joint_3" />
-    <joint name="${tf_prefix}joint_4" />
-    <joint name="${tf_prefix}joint_5" />
-    <joint name="${tf_prefix}joint_6" />
-    <joint name="${tf_prefix}ee_joint" />
-  </group>
+      <chain base_link="${tf_prefix}base_link" tip_link="${tf_prefix}ee_link" />
+    </group>
     <!-- Sub-group for wrist-only control. -->
     <group name="ar_wrist">
-      <joint name="${tf_prefix}joint_6" />
-      <joint name="${tf_prefix}ee_joint"/>
+      <chain base_link="${tf_prefix}link_5" tip_link="${tf_prefix}ee_link" />
     </group>
     <group_state name="home" group="ar_manipulator">

Commit message: simplifying IK by building groups_didn't work

File: ros2_ws/src/james_description/srdf/ar_macro.srdf.xacro (robot description, xacro)
@@ -17,9 +17,14 @@
     <!-- Sub-group for stable cartesian translation (X, Y, Z). Locks J4 and J6. -->
     <group name="ar_translator">
-      <chain base_link="${tf_prefix}base_link" tip_link="${tf_prefix}ee_link" />
+      <joint name="${tf_prefix}joint_1" />
+      <joint name="${tf_prefix}joint_2" />
+      <joint name="${tf_prefix}joint_3" />
+      <joint name="${tf_prefix}joint_5" />
+      <joint name="${tf_prefix}ee_joint"/>
     </group>
     <!-- Sub-group for wrist-only control. -->
     <group name="ar_wrist">
-      <chain base_link="${tf_prefix}link_5" tip_link="${tf_prefix}ee_link" />
+      <joint name="${tf_prefix}joint_6" />
+      <joint name="${tf_prefix}ee_joint"/>
     </group>
     <group_state name="home" group="ar_manipulator">

Commit message: changng approach2

File: ros2_ws/src/james_description/srdf/ar_macro.srdf.xacro (robot description, xacro)
@@ -17,4 +17,12 @@
     <!-- Sub-group for stable cartesian translation (X, Y, Z). Locks J4 and J6. -->
     <group name="ar_translator">
+      <link name="${tf_prefix}base_link" />
+      <link name="${tf_prefix}link_1" />
+      <link name="${tf_prefix}link_2" />
+      <link name="${tf_prefix}link_3" />
+      <link name="${tf_prefix}link_4" />
+      <link name="${tf_prefix}link_5" />
+      <link name="${tf_prefix}link_6" />
+      <link name="${tf_prefix}ee_link" />
       <joint name="${tf_prefix}joint_1" />
       <joint name="${tf_prefix}joint_2" />

Commit message: reversing changes2

File: ros2_ws/src/james_description/srdf/ar_macro.srdf.xacro (robot description, xacro)
@@ -17,12 +17,4 @@
     <!-- Sub-group for stable cartesian translation (X, Y, Z). Locks J4 and J6. -->
     <group name="ar_translator">
-      <link name="${tf_prefix}base_link" />
-      <link name="${tf_prefix}link_1" />
-      <link name="${tf_prefix}link_2" />
-      <link name="${tf_prefix}link_3" />
-      <link name="${tf_prefix}link_4" />
-      <link name="${tf_prefix}link_5" />
-      <link name="${tf_prefix}link_6" />
-      <link name="${tf_prefix}ee_link" />
       <joint name="${tf_prefix}joint_1" />
       <joint name="${tf_prefix}joint_2" />

Commit message: MoveIt Servo Integration simplified testing_v2

File: ros2_ws/src/james_description/srdf/ar_macro.srdf.xacro (robot description, xacro)
@@ -20,9 +20,16 @@
       <joint name="${tf_prefix}joint_2" />
       <joint name="${tf_prefix}joint_3" />
+      <joint name="${tf_prefix}joint_4" />
       <joint name="${tf_prefix}joint_5" />
+      <joint name="${tf_prefix}joint_6" />
       <joint name="${tf_prefix}ee_joint"/>
     </group>
     <!-- Sub-group for wrist-only control. -->
     <group name="ar_wrist">
+      <joint name="${tf_prefix}joint_1" />
+      <joint name="${tf_prefix}joint_2" />
+      <joint name="${tf_prefix}joint_3" />
+      <joint name="${tf_prefix}joint_4" />
+      <joint name="${tf_prefix}joint_5" />
       <joint name="${tf_prefix}joint_6" />
       <joint name="${tf_prefix}ee_joint"/>
